Commit message: add: pyexplore

File: src/beetlebot_description/urdf/beetlebot.xacro (robot description, xacro)
@@ -1,7 +1,45 @@
 <?xml version='1.0' encoding='utf-8'?>
 <robot name="beetlebot" xmlns:xacro="http://www.ros.org/wiki/xacro">
+    <xacro:arg name="namespace" default="" />
+    <xacro:property name="namespace" value="$(arg namespace)" />
     <xacro:include filename="$(find beetlebot_description)/urdf/beetlebot.gazebo" />
+    <material name="base_link_material">
+        <color rgba="0.033104766565152086 0.46778379610254284 0.12477181755144427 1" />
+    </material>
+    <material name="wheel_right_material">
+        <color rgba="0.6375968739867731 0.04373502925049377 0.008023192982520563 1" />
+    </material>
+    <material name="wheel_left_material">
+        <color rgba="0.6375968739867731 0.04373502925049377 0.008023192982520563 1" />
+    </material>
+    <material name="top_base_material">
+        <color rgba="0.033104766565152086 0.46778379610254284 0.12477181755144427 1" />
+    </material>
+    <material name="front_caster_material">
+        <color rgba="0.10702310296918527 0.0069954101845983935 0.3371636150376657 1" />
+    </material>
+    <material name="rear_caster_material">
+        <color rgba="0.10702310296918527 0.0069954101845983935 0.3371636150376657 1" />
+    </material>
+    <material name="right_bar_material">
+        <color rgba="0.23839757380151394 0.12743768042608497 0.7529422167708612 1" />
+    </material>
+    <material name="left_bar_material">
+        <color rgba="0.23839757380151394 0.12743768042608497 0.7529422167708612 1" />
+    </material>
+    <material name="rear_bar_material">
+        <color rgba="0.23839757380151394 0.12743768042608497 0.7529422167708612 1" />
+    </material>
+    <material name="lidar_material">
+        <color rgba="0 0 0 1" />
+    </material>
+    <material name="camera_material">
+        <color rgba="0.015996293361446288 0.22696587349938613 0.07036009568874305 1" />
+    </material>
+    <material name="imu_material">
+        <color rgba="0.25 0.33 0.33 1" />
+    </material>
     <!-- Base Link -->
-    <link name="base_link">
+    <link name="${namespace}base_link">
         <visual>
             <origin xyz="0 0 0" rpy="0 0 0" />
@@ -9,7 +47,5 @@
                 <cylinder radius="0.3" length="0.1" />
             </geometry>
-            <material name="base_link_material">
-                <color rgba="0.033104766565152086 0.46778379610254284 0.12477181755144427 1" />
-            </material>
+            <material name="base_link_material" />
         </visual>
         <collision>
@@ -26,5 +62,5 @@
     </link>
     <!-- Right Wheel Link -->
-    <link name="wheel_right">
+    <link name="${namespace}wheel_right">
         <visual>
             <origin xyz="0 0 0" rpy="0 0 0" />
@@ -32,7 +68,5 @@
                 <cylinder radius="0.15" length="0.07" />
             </geometry>
-            <material name="wheel_right_material">
-                <color rgba="0.6375968739867731 0.04373502925049377 0.008023192982520563 1" />
-            </material>
+            <material name="wheel_right_material" />
         </visual>
         <collision>
@@ -50,12 +84,12 @@
     </link>
     <!-- Right Wheel Joint -->
-    <joint name="base_link_to_wheel_right" type="continuous">
-        <parent link="base_link" />
-        <child link="wheel_right" />
+    <joint name="${namespace}base_link_to_wheel_right" type="continuous">
+        <parent link="${namespace}base_link" />
+        <child link="${namespace}wheel_right" />
         <origin xyz="0 -0.33 -0.05" rpy="1.5707963267948963 0 0" />
         <axis xyz="0 0 -1" />
     </joint>
     <!-- Left Wheel Link -->
-    <link name="wheel_left">
+    <link name="${namespace}wheel_left">
         <visual>
             <origin xyz="0 0 0" rpy="0 0 0" />
@@ -63,7 +97,5 @@
                 <cylinder radius="0.15" length="0.07" />
             </geometry>
-            <material name="wheel_left_material">
-                <color rgba="0.6375968739867731 0.04373502925049377 0.008023192982520563 1" />
-            </material>
+            <material name="wheel_left_material" />
         </visual>
         <collision>
@@ -81,12 +113,12 @@
     </link>
     <!-- Left Wheel Joint -->
-    <joint name="base_link_to_wheel_left" type="continuous">
-        <parent link="base_link" />
-        <child link="wheel_left" />
+    <joint name="${namespace}base_link_to_wheel_left" type="continuous">
+        <parent link="${namespace}base_link" />
+        <child link="${namespace}wheel_left" />
         <origin xyz="0 0.33 -0.05" rpy="1.5707963267948963 0 0" />
         <axis xyz="0 0 -1" />
     </joint>
     <!-- Top Base Link -->
-    <link name="top_base">
+    <link name="${namespace}top_base">
         <visual>
             <origin xyz="0 0 0" rpy="0 0 0" />
@@ -94,7 +126,5 @@
                 <cylinder radius="0.3" length="0.1" />
             </geometry>
-            <material name="top_base_material">
-                <color rgba="0.033104766565152086 0.46778379610254284 0.12477181755144427 1" />
-            </material>
+            <material name="top_base_material" />
         </visual>
         <collision>
@@ -112,11 +142,11 @@
     </link>
     <!-- Top Base Joint -->
-    <joint name="base_link_to_top_base" type="fixed">
-        <parent link="base_link" />
-        <child link="top_base" />
+    <joint name="${namespace}base_link_to_top_base" type="fixed">
+        <parent link="${namespace}base_link" />
+        <child link="${namespace}top_base" />
         <origin xyz="0 0 0.45" rpy="0 0 0" />
     </joint>
     <!-- Front Caster Link -->
-    <link name="front_caster">
+    <link name="${namespace}front_caster">
         <visual>
             <origin xyz="0 0 0" rpy="0 0 0" />
@@ -124,7 +154,5 @@
                 <sphere radius="0.1" />
             </geometry>
-            <material name="front_caster_material">
-                <color rgba="0.10702310296918527 0.0069954101845983935 0.3371636150376657 1" />
-            </material>
+            <material name="front_caster_material" />
         </visual>
         <collision>
@@ -142,12 +170,12 @@
     </link>
     <!-- Front Caster Joint -->
-    <joint name="base_link_to_front_caster" type="fixed">
-        <parent link="base_link" />
-        <child link="front_caster" />
+    <joint name="${namespace}base_link_to_front_caster" type="fixed">
+        <parent link="${namespace}base_link" />
+        <child link="${namespace}front_caster" />
         <origin xyz="0.2 0 -0.1" rpy="0 0 0" />
         <axis xyz="0 1 0" />
     </joint>
     <!-- Rear Caster Link -->
-    <link name="rear_caster">
+    <link name="${namespace}rear_caster">
         <visual>
             <origin xyz="0 0 0" rpy="0 0 0" />
@@ -155,7 +183,5 @@
                 <sphere radius="0.1" />
             </geometry>
-            <material name="rear_caster_material">
-                <color rgba="0.10702310296918527 0.0069954101845983935 0.3371636150376657 1" />
-            </material>
+            <material name="rear_caster_material" />
         </visual>
         <collision>
@@ -172,20 +198,18 @@
     </link>
     <!-- Rear Caster Joint -->
-    <joint name="base_link_to_rear_caster" type="fixed">
-        <parent link="base_link" />
-        <child link="rear_caster" />
+    <joint name="${namespace}base_link_to_rear_caster" type="fixed">
+        <parent link="${namespace}base_link" />
+        <child link="${namespace}rear_caster" />
         <origin xyz="-0.2 0 -0.1" rpy="0 0 0" />
         <axis xyz="0 1 0" />
     </joint>
     <!-- Right Bar Link -->
-    <link name="right_bar">
-        <visual>
-            <origin xyz="0 0 0" rpy="0 0 0" />
-            <geometry>
-                <cylinder radius="0.03" length="0.5" />
-            </geometry>
-            <material name="right_bar_material">
-                <color rgba="0.23839757380151394 0.12743768042608497 0.7529422167708612 1" />
-            </material>
+    <link name="${namespace}right_bar">
+        <visual>
+            <origin xyz="0 0 0" rpy="0 0 0" />
+            <geometry>
+                <cylinder radius="0.03" length="0.5" />
+            </geometry>
+            <material name="right_bar_material" />
         </visual>
         <collision>
@@ -203,19 +227,17 @@
     </link>
     <!-- Right Bar Joint -->
-    <joint name="base_link_to_right_bar" type="fixed">
-        <parent link="base_link" />
-        <child link="right_bar" />
+    <joint name="${namespace}base_link_to_right_bar" type="fixed">
+        <parent link="${namespace}base_link" />
+        <child link="${namespace}right_bar" />
         <origin xyz="0 0.2 0.2058808723746403" rpy="0 0 0" />
     </joint>
     <!-- Left Bar Link -->
-    <link name="left_bar">
-        <visual>
-            <origin xyz="0 0 0" rpy="0 0 0" />
-            <geometry>
-                <cylinder radius="0.03" length="0.5" />
-            </geometry>
-            <material name="left_bar_material">
-                <color rgba="0.23839757380151394 0.12743768042608497 0.7529422167708612 1" />
-            </material>
+    <link name="${namespace}left_bar">
+        <visual>
+            <origin xyz="0 0 0" rpy="0 0 0" />
+            <geometry>
+                <cylinder radius="0.03" length="0.5" />
+            </geometry>
+            <material name="left_bar_material" />
         </visual>
         <collision>
@@ -233,19 +255,17 @@
     </link>
     <!-- Left Bar Joint -->
-    <joint name="base_link_to_left_bar" type="fixed">
-        <parent link="base_link" />
-        <child link="left_bar" />
+    <joint name="${namespace}base_link_to_left_bar" type="fixed">
+        <parent link="${namespace}base_link" />
+        <child link="${namespace}left_bar" />
         <origin xyz="0 -0.2 0.2058808723746403" rpy="0 0 0" />
     </joint>
     <!-- Rear Bar Link -->
-    <link name="rear_bar">
-        <visual>
-            <origin xyz="0 0 0" rpy="0 0 0" />
-            <geometry>
-                <cylinder radius="0.03" length="0.5" />
-            </geometry>
-            <material name="rear_bar_material">
-                <color rgba="0.23839757380151394 0.12743768042608497 0.7529422167708612 1" />
-            </material>
+    <link name="${namespace}rear_bar">
+        <visual>
+            <origin xyz="0 0 0" rpy="0 0 0" />
+            <geometry>
+                <cylinder radius="0.03" length="0.5" />
+            </geometry>
+            <material name="rear_bar_material" />
         </visual>
         <collision>
@@ -263,11 +283,11 @@
     </link>
     <!-- Rear Bar Joint -->
-    <joint name="base_link_to_rear_bar" type="fixed">
-        <parent link="base_link" />
-        <child link="rear_bar" />
+    <joint name="${namespace}base_link_to_rear_bar" type="fixed">
+        <parent link="${namespace}base_link" />
+        <child link="${namespace}rear_bar" />
         <origin xyz="-0.2 0 0.2058808723746403" rpy="0 0 0" />
     </joint>
     <!-- Lidar Link -->
-    <link name="lidar_link">
+    <link name="${namespace}lidar">
         <visual>
             <origin xyz="0 0 0" rpy="0 0 0" />
@@ -275,7 +295,5 @@
                 <cylinder radius="0.1" length="0.13538975482266932" />
             </geometry>
-            <material name="lidar_material">
-                <color rgba="0 0 0 1" />
-            </material>
+            <material name="lidar_material" />
         </visual>
         <collision>
@@ -293,11 +311,11 @@
     </link>
     <!-- Lidar Joint -->
-    <joint name="base_link_to_lidar" type="fixed">
-        <parent link="base_link" />
-        <child link="lidar_link" />
+    <joint name="${namespace}base_link_to_lidar" type="fixed">
+        <parent link="${namespace}base_link" />
+        <child link="${namespace}lidar" />
         <origin xyz="0 0 0.57" rpy="0 0 0" />
     </joint>
     <!-- Camera Link -->
-    <link name="camera_link">
+    <link name="${namespace}camera">
         <visual>
             <origin xyz="0 0 0" rpy="0 0 0" />
@@ -305,7 +323,5 @@
                 <box size="0.05 0.2 0.1" />
             </geometry>
-            <material name="camera_material">
-                <color rgba="0.015996293361446288 0.22696587349938613 0.07036009568874305 1" />
-            </material>
+            <material name="camera_material" />
         </visual>
         <collision>
@@ -323,12 +339,12 @@
     </link>
     <!-- Camera Joint -->
-    <joint name="base_link_to_camera" type="revolute">
-        <parent link="base_link" />
-        <child link="camera_link" />
+    <joint name="${namespace}base_link_to_camera" type="revolute">
+        <parent link="${namespace}base_link" />
+        <child link="${namespace}camera" />
         <origin xyz="0.3 0 0.34" rpy="0 0 0" />
         <axis xyz="0 1 0" />
         <limit lower="-1.14" upper="1.14" velocity="3.14" effort="10.0" />
     </joint>
-    <link name="imu_link">
+    <link name="${namespace}imu_link">
         <visual>
             <origin xyz="0 0 0" rpy="0 0 0" />
@@ -336,7 +352,5 @@
                 <cylinder radius="0.05" length="0.135" />
             </geometry>
-            <material name="imu_material">
-                <color rgba="0.25 0.33 0.33 1" />
-            </material>
+            <material name="imu_material" />
         </visual>
         <collision>
@@ -352,10 +366,10 @@
         </inertial>
     </link>
-    <joint name="base_link_to_imu" type="fixed">
-        <parent link="base_link" />
-        <child link="imu_link" />
+    <joint name="${namespace}base_link_to_imu" type="fixed">
+        <parent link="${namespace}base_link" />
+        <child link="${namespace}imu_link" />
         <origin xyz="0 0 0.1" rpy="0 0 0" />
     </joint>
-    <gazebo reference="imu_link">
+    <gazebo reference="${namespace}imu_link">
         <sensor name="imu_sensor" type="imu">
             <ignition_frame_id>imu_link</ignition_frame_id>

Commit message: fix: odom tf issue

File: src/beetlebot_description/urdf/beetlebot.xacro (robot description, xacro)
@@ -41,5 +41,5 @@
     </material>
     <!-- Base Link -->
-    <link name="${namespace}base_link">
+    <link name="base_link">
         <visual>
             <origin xyz="0 0 0" rpy="0 0 0" />
@@ -62,5 +62,5 @@
     </link>
     <!-- Right Wheel Link -->
-    <link name="${namespace}wheel_right">
+    <link name="wheel_right">
         <visual>
             <origin xyz="0 0 0" rpy="0 0 0" />
@@ -84,12 +84,12 @@
     </link>
     <!-- Right Wheel Joint -->
-    <joint name="${namespace}base_link_to_wheel_right" type="continuous">
-        <parent link="${namespace}base_link" />
-        <child link="${namespace}wheel_right" />
+    <joint name="base_link_to_wheel_right" type="continuous">
+        <parent link="base_link" />
+        <child link="wheel_right" />
         <origin xyz="0 -0.33 -0.05" rpy="1.5707963267948963 0 0" />
         <axis xyz="0 0 -1" />
     </joint>
     <!-- Left Wheel Link -->
-    <link name="${namespace}wheel_left">
+    <link name="wheel_left">
         <visual>
             <origin xyz="0 0 0" rpy="0 0 0" />
@@ -113,12 +113,12 @@
     </link>
     <!-- Left Wheel Joint -->
-    <joint name="${namespace}base_link_to_wheel_left" type="continuous">
-        <parent link="${namespace}base_link" />
-        <child link="${namespace}wheel_left" />
+    <joint name="base_link_to_wheel_left" type="continuous">
+        <parent link="base_link" />
+        <child link="wheel_left" />
         <origin xyz="0 0.33 -0.05" rpy="1.5707963267948963 0 0" />
         <axis xyz="0 0 -1" />
     </joint>
     <!-- Top Base Link -->
-    <link name="${namespace}top_base">
+    <link name="top_base">
         <visual>
             <origin xyz="0 0 0" rpy="0 0 0" />
@@ -142,11 +142,11 @@
     </link>
     <!-- Top Base Joint -->
-    <joint name="${namespace}base_link_to_top_base" type="fixed">
-        <parent link="${namespace}base_link" />
-        <child link="${namespace}top_base" />
+    <joint name="base_link_to_top_base" type="fixed">
+        <parent link="base_link" />
+        <child link="top_base" />
         <origin xyz="0 0 0.45" rpy="0 0 0" />
     </joint>
     <!-- Front Caster Link -->
-    <link name="${namespace}front_caster">
+    <link name="front_caster">
         <visual>
             <origin xyz="0 0 0" rpy="0 0 0" />
@@ -170,12 +170,12 @@
     </link>
     <!-- Front Caster Joint -->
-    <joint name="${namespace}base_link_to_front_caster" type="fixed">
-        <parent link="${namespace}base_link" />
-        <child link="${namespace}front_caster" />
+    <joint name="base_link_to_front_caster" type="fixed">
+        <parent link="base_link" />
+        <child link="front_caster" />
         <origin xyz="0.2 0 -0.1" rpy="0 0 0" />
         <axis xyz="0 1 0" />
     </joint>
     <!-- Rear Caster Link -->
-    <link name="${namespace}rear_caster">
+    <link name="rear_caster">
         <visual>
             <origin xyz="0 0 0" rpy="0 0 0" />
@@ -198,12 +198,12 @@
     </link>
     <!-- Rear Caster Joint -->
-    <joint name="${namespace}base_link_to_rear_caster" type="fixed">
-        <parent link="${namespace}base_link" />
-        <child link="${namespace}rear_caster" />
+    <joint name="base_link_to_rear_caster" type="fixed">
+        <parent link="base_link" />
+        <child link="rear_caster" />
         <origin xyz="-0.2 0 -0.1" rpy="0 0 0" />
         <axis xyz="0 1 0" />
     </joint>
     <!-- Right Bar Link -->
-    <link name="${namespace}right_bar">
+    <link name="right_bar">
         <visual>
             <origin xyz="0 0 0" rpy="0 0 0" />
@@ -227,11 +227,11 @@
     </link>
     <!-- Right Bar Joint -->
-    <joint name="${namespace}base_link_to_right_bar" type="fixed">
-        <parent link="${namespace}base_link" />
-        <child link="${namespace}right_bar" />
+    <joint name="base_link_to_right_bar" type="fixed">
+        <parent link="base_link" />
+        <child link="right_bar" />
         <origin xyz="0 0.2 0.2058808723746403" rpy="0 0 0" />
     </joint>
     <!-- Left Bar Link -->
-    <link name="${namespace}left_bar">
+    <link name="left_bar">
         <visual>
             <origin xyz="0 0 0" rpy="0 0 0" />
@@ -255,11 +255,11 @@
     </link>
     <!-- Left Bar Joint -->
-    <joint name="${namespace}base_link_to_left_bar" type="fixed">
-        <parent link="${namespace}base_link" />
-        <child link="${namespace}left_bar" />
+    <joint name="base_link_to_left_bar" type="fixed">
+        <parent link="base_link" />
+        <child link="left_bar" />
         <origin xyz="0 -0.2 0.2058808723746403" rpy="0 0 0" />
     </joint>
     <!-- Rear Bar Link -->
-    <link name="${namespace}rear_bar">
+    <link name="rear_bar">
         <visual>
             <origin xyz="0 0 0" rpy="0 0 0" />
@@ -283,11 +283,11 @@
     </link>
     <!-- Rear Bar Joint -->
-    <joint name="${namespace}base_link_to_rear_bar" type="fixed">
-        <parent link="${namespace}base_link" />
-        <child link="${namespace}rear_bar" />
+    <joint name="base_link_to_rear_bar" type="fixed">
+        <parent link="base_link" />
+        <child link="rear_bar" />
         <origin xyz="-0.2 0 0.2058808723746403" rpy="0 0 0" />
     </joint>
     <!-- Lidar Link -->
-    <link name="${namespace}lidar">
+    <link name="lidar">
         <visual>
             <origin xyz="0 0 0" rpy="0 0 0" />
@@ -311,11 +311,11 @@
     </link>
     <!-- Lidar Joint -->
-    <joint name="${namespace}base_link_to_lidar" type="fixed">
-        <parent link="${namespace}base_link" />
-        <child link="${namespace}lidar" />
+    <joint name="base_link_to_lidar" type="fixed">
+        <parent link="base_link" />
+        <child link="lidar" />
         <origin xyz="0 0 0.57" rpy="0 0 0" />
     </joint>
     <!-- Camera Link -->
-    <link name="${namespace}camera">
+    <link name="camera">
         <visual>
             <origin xyz="0 0 0" rpy="0 0 0" />
@@ -339,12 +339,12 @@
     </link>
     <!-- Camera Joint -->
-    <joint name="${namespace}base_link_to_camera" type="revolute">
-        <parent link="${namespace}base_link" />
-        <child link="${namespace}camera" />
+    <joint name="base_link_to_camera" type="revolute">
+        <parent link="base_link" />
+        <child link="camera" />
         <origin xyz="0.3 0 0.34" rpy="0 0 0" />
         <axis xyz="0 1 0" />
         <limit lower="-1.14" upper="1.14" velocity="3.14" effort="10.0" />
     </joint>
-    <link name="${namespace}imu_link">
+    <link name="imu_link">
         <visual>
             <origin xyz="0 0 0" rpy="0 0 0" />
@@ -366,15 +366,15 @@
         </inertial>
     </link>
-    <joint name="${namespace}base_link_to_imu" type="fixed">
-        <parent link="${namespace}base_link" />
-        <child link="${namespace}imu_link" />
+    <joint name="base_link_to_imu" type="fixed">
+        <parent link="base_link" />
+        <child link="imu_link" />
         <origin xyz="0 0 0.1" rpy="0 0 0" />
     </joint>
-    <gazebo reference="${namespace}imu_link">
+    <gazebo reference="imu_link">
         <sensor name="imu_sensor" type="imu">
             <ignition_frame_id>imu_link</ignition_frame_id>
             <plugin filename="ignition-gazebo-imu-system" name="ignition::gazebo::systems::Imu">
             </plugin>
-            <topic>imu</topic>
+            <topic>$(arg namespace)imu</topic>
             <always_on>true</always_on>
             <update_rate>100</update_rate>

Commit message: add: pyfrontiers demo-version

File: src/beetlebot_description/urdf/beetlebot.xacro (robot description, xacro)
@@ -295,4 +295,8 @@
                 <cylinder radius="0.1" length="0.13538975482266932" />
             </geometry>
+            <!-- TODO later line 246 - https://github.com/gazebosim/docs/blob/master/fortress/tutorials/spawn_urdf/rrbot.urdf-->
+            <!-- <geometry>
+                <mesh filename="package://rrbot_description/meshes/hokuyo.dae"/>
+            </geometry> -->
             <material name="lidar_material" />
         </visual>
